File: LiDAR-CAN/MCU.kicad_sch (KiCad schematic)
At the start: 25 parts, among them J5 61300511121, SW1 RST, U5 STM32F401RBT6, Y3 25MHz

Commit message: Update complete first placement
Connections:
- net ETHERNET_INT: now also U5.43 (PA10); no longer U5.8 (PC0)
- net ETHERNET_RST: now also U5.42 (PA9); no longer U5.9 (PC1)
Changed lines of the file:
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@@
+	)
+	(no_connect
+		(at 132.08 83.82)
 	)
 	(no_connect
@@
 	)
 	(no_connect
+		(at 132.08 86.36)
+	)
+	(no_connect
 		(at 172.72 119.38)
 	)
@@
 	)
 	(no_connect
-		(at 172.72 81.28)
-	)
-	(no_connect
 		(at 172.72 114.3)
 	)
@@
 	(no_connect
 		(at 132.08 109.22)
-	)
-	(no_connect
-		(at 172.72 78.74)
 	)
 	(no_connect
@@
 		)
 	)
-	(hierarchical_label "ETHERNET_RST"
-		(shape output)
-		(at 132.08 86.36 180)
-		(effects
-			(font
-				(size 1.27 1.27)
-			)
-			(justify right)
-		)
-	)
 	(hierarchical_label "VDD"
 		(shape input)
@@
 		)
 	)
-	(hierarchical_label "ETHERNET_INT"
-		(shape input)
-		(at 132.08 83.82 180)
-		(effects
-			(font
-				(size 1.27 1.27)
-			)
-			(justify right)
-		)
-	)
 	(hierarchical_label "CAN_WKRQ"
 		(shape input)
@@
 		)
 	)
+	(hierarchical_label "ETHERNET_INT"
+		(shape input)
+		(at 172.72 81.28 0)
+		(effects
+			(font
+				(size 1.27 1.27)
+			)
+			(justify left)
+		)
+	)
 	(hierarchical_label "VDD"
 		(shape input)
@@
 		)
 	)
+	(hierarchical_label "ETHERNET_RST"
+		(shape output)
+		(at 172.72 78.74 0)
+		(effects
+			(font
+				(size 1.27 1.27)
+			)
+			(justify left)
+		)
+	)

Commit message: Feature schematic revision 2
Main changes related to connection wires for easy layout and minor components adjustments from Rev 1
Parts:
- J5: Manufacturer Würth Elektronik -> Wurth Elektronik
- R34: value 22Ω -> 22R
Changed lines of the file:
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@@
 	(title_block
 		(title "LiDAR-CAN Interface")
-		(date "2025-08-03")
-		(rev "1")
+		(date "2025-08-05")
+		(rev "2")
 		(company "Robot.com")
 	)
@@
 			)
 		)
-		(property "Manufacturer" "Würth Elektronik"
+		(property "Manufacturer" "Wurth Elektronik"
 			(at 259.08 78.74 0)
 			(effects
@@
 			)
 		)
-		(property "Description" "10 µF ±10% 25V Ceramic Capacitor X5R 0603 (1608 Metric)"
+		(property "Description" "CAP CER 10UF 25V X5R 0603"
 			(at 50.8 44.45 0)
 			(effects
@@
 			)
 		)
-		(property "Value" "22Ω"
+		(property "Value" "22R"
 			(at 44.45 154.94 90)
 			(effects
